File: RTOS Project Schematic/paddle_motors.kicad_sch (KiCad schematic)
At the start: 3 parts, among them M2 Motor_DC, M3 Motor_DC, U3 L298N

Commit message: Added preliminary microphone circuit
Other:
- company: (none) -> Eddie and Felix
- title: (none) -> Paddle Motors
Changed lines of the file:
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@@
 (kicad_sch (version 20230121) (generator eeschema)
   (paper "A4")
+  (title_block
+    (title "Paddle Motors")
+    (date "2023-11-29")
+    (rev "A")
+    (company "Eddie and Felix")
+  )
   (no_connect (at 182.88 107.95))
   (no_connect (at 193.04 72.39))
