File: RTOS Project Schematic/ir_sensor.kicad_sch (KiCad schematic)
At the start: 2 parts

Commit message: Added preliminary microphone circuit
Other:
- company: (none) -> Eddie and Felix
- title: (none) -> IR Beam Sensors
Changed lines of the file:
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@@
 (kicad_sch (version 20230121) (generator eeschema)
   (paper "A4")
+  (title_block
+    (title "IR Beam Sensors")
+    (date "2023-11-29")
+    (rev "A")
+    (company "Eddie and Felix")
+  )
   (junction (at 142.24 73.66) (diameter 0) (color 0 0 0 0)
   )
