File: RTOS Project Schematic/limit_switches.kicad_sch (KiCad schematic)
At the start: 8 parts, among them SW1 SW_SPDT, SW2 SW_SPDT, SW3 SW_SPDT, SW4 SW_SPDT, SW5 SW_SPDT, SW6 SW_SPDT, SW7 SW_SPDT, SW8 SW_SPDT

Commit message: Added preliminary microphone circuit
Other:
- company: (none) -> Eddie and Felix
- title: (none) -> Limit Switches
Changed lines of the file:
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@@
 (kicad_sch (version 20230121) (generator eeschema)
   (paper "A4")
+  (title_block
+    (title "Limit Switches")
+    (date "2023-11-29")
+    (rev "A")
+    (company "Eddie and Felix")
+  )
   (symbol (lib_id "Switch:SW_SPDT") (at 143.51 46.99 0) (unit 1)
     (in_bom yes) (on_board yes) (dnp no) (fields_autoplaced)

Commit message: Updated schematics
Connections:
- net GND: now reaches SW1.2 (B)
- net GND: now also SW2.2 (B), SW3.2 (B), SW4.2 (B), SW5.2 (B), SW6.2 (B)
- net SW1_AL: now reaches SW1.3 (C)
- net SW3_P1L: now reaches SW3.3 (C)
- net SW2_AR: now reaches SW2.3 (C)
- net SW5_P2L: now reaches SW5.3 (C)
- net SW6_P2R: now reaches SW6.3 (C)
- net SW4_P1R: now reaches SW4.3 (C)
Changed lines of the file:
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@@
     (company "Eddie and Felix")
+  )
+  (junction (at 130.81 110.49) (diameter 0) (color 0 0 0 0)
+  )
+  (junction (at 130.81 46.99) (diameter 0) (color 0 0 0 0)
+  )
+  (junction (at 130.81 63.5) (diameter 0) (color 0 0 0 0)
+  )
+  (junction (at 130.81 93.98) (diameter 0) (color 0 0 0 0)
+  )
+  (junction (at 130.81 78.74) (diameter 0) (color 0 0 0 0)
+  )
+  (wire (pts (xy 148.59 49.53) (xy 163.83 49.53))
+    (stroke (width 0) (type default))
+  )
+  (wire (pts (xy 148.59 113.03) (xy 163.83 113.03))
+    (stroke (width 0) (type default))
+  )
+  (wire (pts (xy 138.43 93.98) (xy 130.81 93.98))
+    (stroke (width 0) (type default))
+  )
+  (wire (pts (xy 130.81 93.98) (xy 130.81 78.74))
+    (stroke (width 0) (type default))
+  )
+  (wire (pts (xy 138.43 78.74) (xy 130.81 78.74))
+    (stroke (width 0) (type default))
+  )
+  (wire (pts (xy 130.81 78.74) (xy 130.81 63.5))
+    (stroke (width 0) (type default))
+  )
+  (wire (pts (xy 148.59 66.04) (xy 163.83 66.04))
+    (stroke (width 0) (type default))
+  )
+  (wire (pts (xy 138.43 127) (xy 130.81 127))
+    (stroke (width 0) (type default))
+  )
+  (wire (pts (xy 148.59 129.54) (xy 163.83 129.54))
+    (stroke (width 0) (type default))
+  )
+  (wire (pts (xy 130.81 63.5) (xy 130.81 46.99))
+    (stroke (width 0) (type default))
+  )
+  (wire (pts (xy 138.43 110.49) (xy 130.81 110.49))
+    (stroke (width 0) (type default))
+  )
+  (wire (pts (xy 130.81 110.49) (xy 130.81 93.98))
+    (stroke (width 0) (type default))
+  )
+  (wire (pts (xy 130.81 127) (xy 130.81 110.49))
+    (stroke (width 0) (type default))
+  )
+  (wire (pts (xy 130.81 46.99) (xy 138.43 46.99))
+    (stroke (width 0) (type default))
+  )
+  (wire (pts (xy 138.43 63.5) (xy 130.81 63.5))
+    (stroke (width 0) (type default))
+  )
+  (wire (pts (xy 93.98 46.99) (xy 130.81 46.99))
+    (stroke (width 0) (type default))
+  )
+  (wire (pts (xy 148.59 81.28) (xy 163.83 81.28))
+    (stroke (width 0) (type default))
+  )
+  (wire (pts (xy 148.59 96.52) (xy 163.83 96.52))
+    (stroke (width 0) (type default))
+  )
+  (hierarchical_label "SW3_P1L" (shape output) (at 163.83 81.28 0) (fields_autoplaced)
+    (effects (font (size 1.27 1.27)) (justify left))
+  )
+  (hierarchical_label "SW6_P2R" (shape output) (at 163.83 129.54 0) (fields_autoplaced)
+    (effects (font (size 1.27 1.27)) (justify left))
+  )
+  (hierarchical_label "SW1_AL" (shape output) (at 163.83 49.53 0) (fields_autoplaced)
+    (effects (font (size 1.27 1.27)) (justify left))
+  )
+  (hierarchical_label "SW4_P1R" (shape output) (at 163.83 96.52 0) (fields_autoplaced)
+    (effects (font (size 1.27 1.27)) (justify left))
+  )
+  (hierarchical_label "SW5_P2L" (shape output) (at 163.83 113.03 0) (fields_autoplaced)
+    (effects (font (size 1.27 1.27)) (justify left))
+  )
+  (hierarchical_label "GND" (shape input) (at 93.98 46.99 180) (fields_autoplaced)
+    (effects (font (size 1.27 1.27)) (justify right))
+  )
+  (hierarchical_label "SW2_AR" (shape output) (at 163.83 66.04 0) (fields_autoplaced)
+    (effects (font (size 1.27 1.27)) (justify left))
   )
   (symbol (lib_id "Switch:SW_SPDT") (at 143.51 46.99 0) (unit 1)
