File: RTOS Project Schematic/tilt_motor.kicad_sch (KiCad schematic)
At the start: 3 parts, among them M1 NEMA-17 STEPPER MOTOR

Commit message: Added preliminary microphone circuit
Parts:
- C1: value C -> 100u
Other:
- company: (none) -> Eddie and Felix
- title: (none) -> Tilt Motor
Changed lines of the file:
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@@
 (kicad_sch (version 20230121) (generator eeschema)
   (paper "A4")
+  (title_block
+    (title "Tilt Motor")
+    (date "2023-11-29")
+    (rev "A")
+    (company "Eddie and Felix")
+  )
   (junction (at 173.99 106.68) (diameter 0) (color 0 0 0 0)
   )
@@
       (effects (font (size 1.27 1.27)) (justify left))
     )
-    (property "Value" "C" (at 111.76 85.09 0)
-      (effects (font (size 1.27 1.27)) (justify left))
-    )
+    (property "Value" "100u" (at 111.76 85.09 0)
+      (effects (font (size 1.27 1.27)) (justify left))
+    )
