File: RTOS Project Schematic/RTOS Project Schematic.kicad_sch (KiCad schematic)
At the start: 0 parts

Commit message: Updated schematic
Other:
- sheet LCD ports: added GND, SCL, SDA, VCC; removed none
- sheet Raspberry Pi ports: added 3V3_LCD, GND_LCD, I2C_SCL, I2C_SDA, SPI_MISO; removed SPI_SIMO
Changed lines of the file:
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@@
+    (stroke (width 0) (type default))
+  )
+  (wire (pts (xy 208.28 38.1) (xy 233.68 38.1))
     (stroke (width 0) (type default))
   )
@@
     (stroke (width 0) (type default))
   )
+  (wire (pts (xy 208.28 48.26) (xy 233.68 48.26))
+    (stroke (width 0) (type default))
+  )
   (wire (pts (xy 233.68 114.3) (xy 173.99 114.3))
     (stroke (width 0) (type default))
@@
     (stroke (width 0) (type default))
   )
+  (wire (pts (xy 208.28 34.29) (xy 233.68 34.29))
+    (stroke (width 0) (type default))
+  )
   (wire (pts (xy 173.99 114.3) (xy 173.99 149.86))
     (stroke (width 0) (type default))
   )
+  (wire (pts (xy 208.28 45.72) (xy 233.68 45.72))
+    (stroke (width 0) (type default))
+  )
   (wire (pts (xy 78.74 41.91) (xy 78.74 73.66))
     (stroke (width 0) (type default))
@@
     (stroke (width 0) (type default))
   )
-  (sheet (at 45.72 120.65) (size 20.32 29.21) (fields_autoplaced)
-    (stroke (width 0.1524) (type solid))
-    (fill (color 0 0 0 0.0000))
-    (property "Sheetname" "LCD" (at 45.72 119.9384 0)
-      (effects (font (size 1.27 1.27)) (justify left bottom))
-    )
-    (property "Sheetfile" "lcd.kicad_sch" (at 45.72 150.4446 0)
-      (effects (font (size 1.27 1.27)) (justify left top))
+  (sheet (at 233.68 30.48) (size 20.32 20.32) (fields_autoplaced)
+    (stroke (width 0.1524) (type solid))
+    (fill (color 0 0 0 0.0000))
+    (property "Sheetname" "LCD" (at 233.68 29.7684 0)
+      (effects (font (size 1.27 1.27)) (justify left bottom))
+    )
+    (property "Sheetfile" "lcd.kicad_sch" (at 233.68 51.3846 0)
+      (effects (font (size 1.27 1.27)) (justify left top))
+    )
+    (pin "GND" input (at 233.68 38.1 180)
+      (effects (font (size 1.27 1.27)) (justify left))
+    )
+    (pin "VCC" input (at 233.68 34.29 180)
+      (effects (font (size 1.27 1.27)) (justify left))
+    )
+    (pin "SDA" input (at 233.68 45.72 180)
+      (effects (font (size 1.27 1.27)) (justify left))
+    )
+    (pin "SCL" input (at 233.68 48.26 180)
+      (effects (font (size 1.27 1.27)) (justify left))
     )
     (instances
@@
       (effects (font (size 1.27 1.27)) (justify left))
     )
-    (pin "SPI_SIMO" bidirectional (at 179.07 50.8 180)
-      (effects (font (size 1.27 1.27)) (justify left))
-    )
     (pin "SPI_CLK" bidirectional (at 179.07 45.72 180)
       (effects (font (size 1.27 1.27)) (justify left))
@@
       (effects (font (size 1.27 1.27)) (justify left))
     )
-    (instances
+    (pin "3V3_LCD" output (at 208.28 34.29 0)
+      (effects (font (size 1.27 1.27)) (justify right))
+    )
+    (pin "GND_LCD" output (at 208.28 38.1 0)
+      (effects (font (size 1.27 1.27)) (justify right))
+    )
+    (pin "SPI_MISO" bidirectional (at 179.07 50.8 180)
+      (effects (font (size 1.27 1.27)) (justify left))
+    )
+    (pin "I2C_SDA" output (at 208.28 45.72 0)
+      (effects (font (size 1.27 1.27)) (justify right))
+    )
+    (pin "I2C_SCL" output (at 208.28 48.26 0)
+      (effects (font (size 1.27 1.27)) (justify right))
+    )
+    (instances
