File: RTOS Project Schematic/lcd.kicad_sch (KiCad schematic)
At the start: 0 parts

Commit message: Updated schematic
Parts:
- added J10: Conn_01x04_Pin, symbol Connector:Conn_01x04_Pin
Connections:
- new net GND: J10.1 (GND)
- new net SCL: J10.4 (SCL)
- new net SDA: J10.3 (SDA)
- new net VCC: J10.2 (VCC)
Changed lines of the file:
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@@
     (company "Eddie and Felix")
   )
+  (wire (pts (xy 147.32 76.2) (xy 162.56 76.2))
+    (stroke (width 0) (type default))
+  )
+  (wire (pts (xy 147.32 68.58) (xy 162.56 68.58))
+    (stroke (width 0) (type default))
+  )
+  (wire (pts (xy 147.32 73.66) (xy 162.56 73.66))
+    (stroke (width 0) (type default))
+  )
+  (wire (pts (xy 147.32 71.12) (xy 162.56 71.12))
+    (stroke (width 0) (type default))
+  )
+  (hierarchical_label "SCL" (shape input) (at 162.56 76.2 0) (fields_autoplaced)
+    (effects (font (size 1.27 1.27)) (justify left))
+  )
+  (hierarchical_label "VCC" (shape input) (at 162.56 71.12 0) (fields_autoplaced)
+    (effects (font (size 1.27 1.27)) (justify left))
+  )
+  (hierarchical_label "SDA" (shape input) (at 162.56 73.66 0) (fields_autoplaced)
+    (effects (font (size 1.27 1.27)) (justify left))
+  )
+  (hierarchical_label "GND" (shape input) (at 162.56 68.58 0) (fields_autoplaced)
+    (effects (font (size 1.27 1.27)) (justify left))
+  )
+  (symbol (lib_id "Connector:Conn_01x04_Pin") (at 142.24 71.12 0) (unit 1)
+    (in_bom yes) (on_board yes) (dnp no) (fields_autoplaced)
+    (property "Reference" "J10" (at 142.875 63.5 0)
+      (effects (font (size 1.27 1.27)))
+    )
+    (property "Value" "Conn_01x04_Pin" (at 142.875 66.04 0)
+      (effects (font (size 1.27 1.27)))
+    )
+    (property "Footprint" "" (at 142.24 71.12 0)
+      (effects (font (size 1.27 1.27)) hide)
+    )
+    (property "Datasheet" "~" (at 142.24 71.12 0)
+      (effects (font (size 1.27 1.27)) hide)
+    )
+    (pin "4")
+    (pin "3")
+    (pin "1")
+    (pin "2")
+    (instances
+      (project "RTOS Project Schematic"
+        (path "/c6d2ace8-9811-4d31-9242-ec8aa6e12e77/2b78a516-d04a-4fbc-85fc-b089c7b78372"
+          (reference "J10") (unit 1)
+        )
+      )
+    )
+  )
 )
