File: RTOS Project Schematic/raspberry_pi.kicad_sch (KiCad schematic)
At the start: 1 part, among them U1 RP2040

Commit message: Added preliminary microphone circuit
Other:
- company: (none) -> Eddie and Felix
- title: (none) -> Raspberry Pi
Changed lines of the file:
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@@
 (kicad_sch (version 20230121) (generator eeschema)
   (paper "A4")
+  (title_block
+    (title "Raspberry Pi")
+    (date "2023-11-29")
+    (rev "A")
+    (company "Eddie and Felix")
+  )
   (wire (pts (xy 118.11 55.88) (xy 118.11 64.77))
     (stroke (width 0) (type default))

Commit message: Updated schematics
Connections:
- net SPI_CLK: now reaches U1.52 (QSPI_SCLK)
Changed lines of the file:
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@@
     (company "Eddie and Felix")
+  )
+  (wire (pts (xy 55.88 105.41) (xy 87.63 105.41))
+    (stroke (width 0) (type default))
   )
   (wire (pts (xy 118.11 55.88) (xy 118.11 64.77))
@@
     (stroke (width 0) (type default))
   )
+  (hierarchical_label "SPI_CLK" (shape bidirectional) (at 55.88 105.41 180) (fields_autoplaced)
+    (effects (font (size 1.27 1.27)) (justify right))
+  )
   (hierarchical_label "GND" (shape input) (at 57.15 161.29 180) (fields_autoplaced)
+    (effects (font (size 1.27 1.27)) (justify right))
+  )
+  (hierarchical_label "SPI_CS" (shape bidirectional) (at 55.88 90.17 180) (fields_autoplaced)
+    (effects (font (size 1.27 1.27)) (justify right))
+  )
+  (hierarchical_label "SPI_SIMO" (shape bidirectional) (at 55.88 97.79 180) (fields_autoplaced)
     (effects (font (size 1.27 1.27)) (justify right))
   )
@@
     (effects (font (size 1.27 1.27)) (justify right))
   )
+  (hierarchical_label "SPI_MOSI" (shape bidirectional) (at 55.88 95.25 180) (fields_autoplaced)
+    (effects (font (size 1.27 1.27)) (justify right))
+  )

Commit message: Updated schematic
Parts:
- added J9: Conn_02x20_Top_Bottom, symbol Connector_Generic:Conn_02x20_Top_Bottom
Connections:
- net SPI_CLK: now also J9.12 (Pin_12); no longer U1.52 (QSPI_SCLK)
- net SPI_CS: now also J9.32 (Pin_32)
- net SPI_MOSI: now also J9.10 (Pin_10)
- new net 3V3_LCD: J9.1 (Pin_1)
- new net GND_LCD: J9.5 (Pin_5)
- new net I2C_SCL: J9.3 (Pin_3)
- new net I2C_SDA: J9.2 (Pin_2)
- new net SPI_MISO: J9.11 (Pin_11)
Other:
- moved on the sheet: U1
Changed lines of the file:
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@@
     (company "Eddie and Felix")
   )
-  (wire (pts (xy 55.88 105.41) (xy 87.63 105.41))
-    (stroke (width 0) (type default))
-  )
-  (wire (pts (xy 118.11 55.88) (xy 118.11 64.77))
-    (stroke (width 0) (type default))
-  )
-  (wire (pts (xy 113.03 161.29) (xy 113.03 156.21))
-    (stroke (width 0) (type default))
-  )
-  (wire (pts (xy 57.15 55.88) (xy 118.11 55.88))
-    (stroke (width 0) (type default))
-  )
-  (wire (pts (xy 57.15 161.29) (xy 113.03 161.29))
-    (stroke (width 0) (type default))
-  )
-  (hierarchical_label "SPI_CLK" (shape bidirectional) (at 55.88 105.41 180) (fields_autoplaced)
-    (effects (font (size 1.27 1.27)) (justify right))
-  )
-  (hierarchical_label "GND" (shape input) (at 57.15 161.29 180) (fields_autoplaced)
-    (effects (font (size 1.27 1.27)) (justify right))
-  )
-  (hierarchical_label "SPI_CS" (shape bidirectional) (at 55.88 90.17 180) (fields_autoplaced)
-    (effects (font (size 1.27 1.27)) (justify right))
-  )
-  (hierarchical_label "SPI_SIMO" (shape bidirectional) (at 55.88 97.79 180) (fields_autoplaced)
-    (effects (font (size 1.27 1.27)) (justify right))
-  )
-  (hierarchical_label "VCC" (shape input) (at 57.15 55.88 180) (fields_autoplaced)
-    (effects (font (size 1.27 1.27)) (justify right))
-  )
-  (hierarchical_label "SPI_MOSI" (shape bidirectional) (at 55.88 95.25 180) (fields_autoplaced)
-    (effects (font (size 1.27 1.27)) (justify right))
-  )
-  (symbol (lib_id "MCU_RaspberryPi:RP2040") (at 113.03 110.49 0) (unit 1)
+  (wire (pts (xy 168.91 87.63) (xy 185.42 87.63))
+    (stroke (width 0) (type default))
+  )
+  (wire (pts (xy 168.91 113.03) (xy 185.42 113.03))
+    (stroke (width 0) (type default))
+  )
+  (wire (pts (xy 168.91 97.79) (xy 185.42 97.79))
+    (stroke (width 0) (type default))
+  )
+  (wire (pts (xy 198.12 115.57) (xy 217.17 115.57))
+    (stroke (width 0) (type default))
+  )
+  (wire (pts (xy 92.71 55.88) (xy 92.71 64.77))
+    (stroke (width 0) (type default))
+  )
+  (wire (pts (xy 168.91 110.49) (xy 185.42 110.49))
+    (stroke (width 0) (type default))
+  )
+  (wire (pts (xy 87.63 161.29) (xy 87.63 156.21))
+    (stroke (width 0) (type default))
+  )
+  (wire (pts (xy 31.75 55.88) (xy 92.71 55.88))
+    (stroke (width 0) (type default))
+  )
+  (wire (pts (xy 168.91 90.17) (xy 185.42 90.17))
+    (stroke (width 0) (type default))
+  )
+  (wire (pts (xy 168.91 92.71) (xy 185.42 92.71))
+    (stroke (width 0) (type default))
+  )
+  (wire (pts (xy 31.75 161.29) (xy 87.63 161.29))
+    (stroke (width 0) (type default))
+  )
+  (wire (pts (xy 168.91 115.57) (xy 185.42 115.57))
+    (stroke (width 0) (type default))
+  )
+  (hierarchical_label "I2C_SCL" (shape output) (at 168.91 92.71 180) (fields_autoplaced)
+    (effects (font (size 1.27 1.27)) (justify right))
+  )
+  (hierarchical_label "SPI_CLK" (shape bidirectional) (at 168.91 115.57 180) (fields_autoplaced)
+    (effects (font (size 1.27 1.27)) (justify right))
+  )
+  (hierarchical_label "GND" (shape input) (at 31.75 161.29 180) (fields_autoplaced)
+    (effects (font (size 1.27 1.27)) (justify right))
+  )
+  (hierarchical_label "SPI_CS" (shape bidirectional) (at 217.17 115.57 0) (fields_autoplaced)
+    (effects (font (size 1.27 1.27)) (justify left))
+  )
+  (hierarchical_label "SPI_MISO" (shape bidirectional) (at 168.91 113.03 180) (fields_autoplaced)
+    (effects (font (size 1.27 1.27)) (justify right))
+  )
+  (hierarchical_label "VCC" (shape input) (at 31.75 55.88 180) (fields_autoplaced)
+    (effects (font (size 1.27 1.27)) (justify right))
+  )
+  (hierarchical_label "GND_LCD" (shape output) (at 168.91 97.79 180) (fields_autoplaced)
+    (effects (font (size 1.27 1.27)) (justify right))
+  )
+  (hierarchical_label "SPI_MOSI" (shape bidirectional) (at 168.91 110.49 180) (fields_autoplaced)
+    (effects (font (size 1.27 1.27)) (justify right))
+  )
+  (hierarchical_label "3V3_LCD" (shape output) (at 168.91 87.63 180) (fields_autoplaced)
+    (effects (font (size 1.27 1.27)) (justify right))
+  )
+  (hierarchical_label "I2C_SDA" (shape output) (at 168.91 90.17 180) (fields_autoplaced)
+    (effects (font (size 1.27 1.27)) (justify right))
+  )
+  (symbol (lib_id "MCU_RaspberryPi:RP2040") (at 87.63 110.49 0) (unit 1)
     (in_bom yes) (on_board yes) (dnp no) (fields_autoplaced)
-    (property "Reference" "U1" (at 115.2241 154.94 0)
+    (property "Reference" "U1" (at 89.8241 154.94 0)
       (effects (font (size 1.27 1.27)) (justify left))
     )
-    (property "Value" "RP2040" (at 115.2241 157.48 0)
+    (property "Value" "RP2040" (at 89.8241 157.48 0)
       (effects (font (size 1.27 1.27)) (justify left))
     )
-    (property "Footprint" "Package_DFN_QFN:QFN-56-1EP_7x7mm_P0.4mm_EP3.2x3.2mm" (at 113.03 110.49 0)
-      (effects (font (size 1.27 1.27)) hide)
-    )
-    (property "Datasheet" "https://datasheets.raspberrypi.com/rp2040/rp2040-datasheet.pdf" (at 113.03 110.49 0)
+    (property "Footprint" "Package_DFN_QFN:QFN-56-1EP_7x7mm_P0.4mm_EP3.2x3.2mm" (at 87.63 110.49 0)
+      (effects (font (size 1.27 1.27)) hide)
+    )
+    (property "Datasheet" "https://datasheets.raspberrypi.com/rp2040/rp2040-datasheet.pdf" (at 87.63 110.49 0)
       (effects (font (size 1.27 1.27)) hide)
     )
@@
         )
       )
+    )
+  )
+  (symbol (lib_id "Connector_Generic:Conn_02x20_Top_Bottom") (at 190.5 110.49 0) (unit 1)
+    (in_bom yes) (on_board yes) (dnp no) (fields_autoplaced)
+    (property "Reference" "J9" (at 191.77 81.28 0)
+      (effects (font (size 1.27 1.27)))
+    )
+    (property "Value" "Conn_02x20_Top_Bottom" (at 191.77 83.82 0)
+      (effects (font (size 1.27 1.27)))
+    )
+    (property "Footprint" "" (at 190.5 110.49 0)
+      (effects (font (size 1.27 1.27)) hide)
+    )
+    (property "Datasheet" "~" (at 190.5 110.49 0)
+      (effects (font (size 1.27 1.27)) hide)
+    )
+    (pin "2")
+    (pin "20")
+    (pin "21")
+    (pin "10")
+    (pin "29")
+    (pin "26")
+    (pin "30")
+    (pin "19")
+    (pin "12")
+    (pin "23")
+    (pin "25")
+    (pin "31")
+    (pin "11")
+    (pin "34")
+    (pin "35")
+    (pin "38")
+    (pin "33")
+    (pin "39")
+    (pin "4")
+    (pin "40")
+    (pin "22")
+    (pin "3")
+    (pin "37")
+    (pin "5")
+    (pin "6")
+    (pin "15")
+    (pin "32")
+    (pin "36")
+    (pin "1")
+    (pin "24")
+    (pin "18")
+    (pin "27")
+    (pin "28")
+    (pin "13")
+    (pin "14")
+    (pin "16")
+    (pin "17")
+    (pin "7")
+    (pin "9")
+    (pin "8")
+    (instances
+      (project "RTOS Project Schematic"
+        (path "/c6d2ace8-9811-4d31-9242-ec8aa6e12e77/c6b733b1-5757-4c9c-9fc9-4998fd29211f"
+          (reference "J9") (unit 1)
+        )
+      )
